File: EnvOpenPico/3V3_power_supply.sch (KiCad schematic (older format))
At the start: 3 parts, among them U2 TLV75533PDBVR

Commit message: Adding parts to pcb
Parts:
- CBP1: footprint Capacitor_SMD:C_0402_1005Metric -> Capacitor_SMD:C_0603_1608Metric
Changed lines of the file:
@@
 F 0 "CBP1" H 5465 3596 50  0000 L CNN
 F 1 "10uf 0402" H 5300 3550 20  0000 L CNN
-F 2 "Capacitor_SMD:C_0402_1005Metric" H 5388 3400 50  0001 C CNN
+F 2 "Capacitor_SMD:C_0603_1608Metric" H 5388 3400 50  0001 C CNN
 F 3 "" H 5350 3550 50  0001 C CNN
 F 4 " " H 5350 3550 50  0001 C CNN "LCSC"

Commit message: Adding Touch
Parts:
- added C60: 10uf 0402, Capacitor_SMD:C_0402_1005Metric, symbol Device:C
- added CBP2: 10uf 0402, Capacitor_SMD:C_0603_1608Metric, symbol Device:C
- added U6: TLV75533PDBVR, Package_TO_SOT_SMD:SOT-23-5, symbol Regulator_Linear:AP131-15
Connections:
- net 5V: now also U6.1 (IN)
- net EN: now also U6.3 (EN)
- net GND: now also C60.2, CBP2.2, U6.2 (GND)
- new net: CBP2.1, U6.4 (BP)
- new net 3V3A: C60.1, U6.5 (OUT)
Changed lines of the file:
@@
 $Descr A4 11693 8268
 encoding utf-8
-Sheet 2 4
+Sheet 2 6
 Title ""
 Date ""
@@
 Text Label 3500 3750 0    50   ~ 0
 3V3_out
+$Comp
+L power:GND #PWR?
+U 1 1 6183D2FC
+P 7400 4050
+AR Path="/6183D2FC" Ref="#PWR?"  Part="1"
+AR Path="/617722D3/6183D2FC" Ref="#PWR076"  Part="1"
+F 0 "#PWR076" H 7400 3800 50  0001 C CNN
+F 1 "GND" H 7405 3877 50  0000 C CNN
+F 2 "" H 7400 4050 50  0001 C CNN
+F 3 "" H 7400 4050 50  0001 C CNN
+	1    7400 4050
+	1    0    0    -1
+$EndComp
+$Comp
+L Device:C C?
+U 1 1 6183D303
+P 8500 3400
+AR Path="/6183D303" Ref="C?"  Part="1"
+AR Path="/617722D3/6183D303" Ref="C60"  Part="1"
+F 0 "C60" H 8615 3446 50  0000 L CNN
+F 1 "10uf 0402" H 8450 3400 20  0000 L CNN
+F 2 "Capacitor_SMD:C_0402_1005Metric" H 8538 3250 50  0001 C CNN
+F 3 "" H 8500 3400 50  0001 C CNN
+F 4 " " H 8500 3400 50  0001 C CNN "LCSC"
+	1    8500 3400
+	1    0    0    -1
+$EndComp
+$Comp
+L power:GND #PWR?
+U 1 1 6183D309
+P 8500 3600
+AR Path="/6183D309" Ref="#PWR?"  Part="1"
+AR Path="/617722D3/6183D309" Ref="#PWR078"  Part="1"
+F 0 "#PWR078" H 8500 3350 50  0001 C CNN
+F 1 "GND" H 8350 3550 50  0000 C CNN
+F 2 "" H 8500 3600 50  0001 C CNN
+F 3 "" H 8500 3600 50  0001 C CNN
+	1    8500 3600
+	1    0    0    -1
+$EndComp
+Wire Wire Line
+	8500 3550 8500 3600
+$Comp
+L Regulator_Linear:AP131-15 U?
+U 1 1 6183D311
+P 7400 3350
+AR Path="/6183D311" Ref="U?"  Part="1"
+AR Path="/617722D3/6183D311" Ref="U6"  Part="1"
+F 0 "U6" H 7400 3692 50  0000 C CNN
+F 1 "TLV75533PDBVR" H 7400 3601 50  0000 C CNN
+F 2 "Package_TO_SOT_SMD:SOT-23-5" H 7400 3675 50  0001 C CIN
+F 3 "" H 7400 3400 50  0001 C CNN
+F 4 " " H 7400 3350 50  0001 C CNN "LCSC"
+	1    7400 3350
+	1    0    0    -1
+$EndComp
+Wire Wire Line
+	7700 3250 8500 3250
+Wire Wire Line
+	7400 3650 7400 4050
+$Comp
+L Device:C CBP?
+U 1 1 6183D31A
+P 7750 3550
+AR Path="/6183D31A" Ref="CBP?"  Part="1"
+AR Path="/617722D3/6183D31A" Ref="CBP2"  Part="1"
+F 0 "CBP2" H 7865 3596 50  0000 L CNN
+F 1 "10uf 0402" H 7700 3550 20  0000 L CNN
+F 2 "Capacitor_SMD:C_0603_1608Metric" H 7788 3400 50  0001 C CNN
+F 3 "" H 7750 3550 50  0001 C CNN
+F 4 " " H 7750 3550 50  0001 C CNN "LCSC"
+	1    7750 3550
+	1    0    0    -1
+$EndComp
+$Comp
+L power:GND #PWR?
+U 1 1 6183D320
+P 7750 3750
+AR Path="/6183D320" Ref="#PWR?"  Part="1"
+AR Path="/617722D3/6183D320" Ref="#PWR077"  Part="1"
+F 0 "#PWR077" H 7750 3500 50  0001 C CNN
+F 1 "GND" H 7600 3700 50  0000 C CNN
+F 2 "" H 7750 3750 50  0001 C CNN
+F 3 "" H 7750 3750 50  0001 C CNN
+	1    7750 3750
+	1    0    0    -1
+$EndComp
+Wire Wire Line
+	7750 3750 7750 3700
+Wire Wire Line
+	7750 3400 7750 3350
+Wire Wire Line
+	7750 3350 7700 3350
+Text Notes 7500 4200 0    50   Italic 0
+Only fit cBP1 if you have selected an \nalternate voltage regulator\n\nTLV75533PDBVR does not.
+Wire Wire Line
+	7100 3250 6750 3250
+Wire Wire Line
+	7100 3350 6750 3350
+Text Label 6750 3250 0    50   ~ 0
+5V_IN
+Text Label 6750 3350 0    50   ~ 0
+Enable
+Text Label 8200 3250 0    50   ~ 0
+3V3A_out
+Text HLabel 3200 3950 0    50   Output ~ 0
+3V3A
+Text Label 3500 3950 0    50   ~ 0
+3V3A_out
+Wire Wire Line
+	3200 3950 3500 3950
 $EndSCHEMATC
