File: EnvOpenPico/DAC.sch (KiCad schematic (older format))
At the start: 36 parts, among them J3 JACK_TRS_6PINS_APPLE, J4 JACK_TRS_6PINS_APPLE, U3 PCM5100, U4 PAM8908

Commit message: Adding Touch
Parts:
- added R26: 0R, Resistor_SMD:R_0402_1005Metric, symbol Device:R_Small
- R13, R14, R15, R16, R17, R18, R19, R20, R21: footprint Capacitor_SMD:C_0402_1005Metric -> Resistor_SMD:R_0402_1005Metric
Connections:
- net GND: now also R26.2
- net GNDA: now also R26.1
Changed lines of the file:
@@
 $Descr A4 11693 8268
 encoding utf-8
-Sheet 3 4
+Sheet 3 6
 Title ""
 Date ""
@@
 F 0 "R15" V 3800 2650 50  0000 C CNN
 F 1 "470" V 3850 2450 50  0000 C CNN
-F 2 "Capacitor_SMD:C_0402_1005Metric" H 3850 2450 50  0001 C CNN
+F 2 "Resistor_SMD:R_0402_1005Metric" H 3850 2450 50  0001 C CNN
 F 3 "~" H 3850 2450 50  0001 C CNN
 	1    3850 2450
@@
 F 0 "R16" V 3900 2750 50  0000 C CNN
 F 1 "470" V 3850 2550 50  0000 C CNN
-F 2 "Capacitor_SMD:C_0402_1005Metric" H 3850 2550 50  0001 C CNN
+F 2 "Resistor_SMD:R_0402_1005Metric" H 3850 2550 50  0001 C CNN
 F 3 "~" H 3850 2550 50  0001 C CNN
 	1    3850 2550
@@
 F 0 "R14" V 1600 3250 50  0000 L CNN
 F 1 "10K" V 1750 3100 50  0000 L CNN
-F 2 "Capacitor_SMD:C_0402_1005Metric" H 1700 3350 50  0001 C CNN
+F 2 "Resistor_SMD:R_0402_1005Metric" H 1700 3350 50  0001 C CNN
 F 3 "~" H 1700 3350 50  0001 C CNN
 	1    1700 3350
@@
 F 0 "R13" V 1550 3150 50  0000 C CNN
 F 1 "5K9" V 1350 3150 50  0000 C CNN
-F 2 "Capacitor_SMD:C_0402_1005Metric" H 1450 3150 50  0001 C CNN
+F 2 "Resistor_SMD:R_0402_1005Metric" H 1450 3150 50  0001 C CNN
 F 3 "~" H 1450 3150 50  0001 C CNN
 	1    1450 3150
@@
 F 0 "R19" V 9700 2300 50  0000 C CNN
 F 1 "33K" V 9800 2300 50  0000 C CNN
-F 2 "Capacitor_SMD:C_0402_1005Metric" H 9800 2300 50  0001 C CNN
+F 2 "Resistor_SMD:R_0402_1005Metric" H 9800 2300 50  0001 C CNN
 F 3 "~" H 9800 2300 50  0001 C CNN
 	1    9800 2300
@@
 F 0 "R18" V 9700 1950 50  0000 C CNN
 F 1 "330" V 9800 1950 50  0000 C CNN
-F 2 "Capacitor_SMD:C_0402_1005Metric" H 9800 1950 50  0001 C CNN
+F 2 "Resistor_SMD:R_0402_1005Metric" H 9800 1950 50  0001 C CNN
 F 3 "~" H 9800 1950 50  0001 C CNN
 	1    9800 1950
@@
 F 0 "R20" V 10300 1950 50  0000 C CNN
 F 1 "330" V 10400 1950 50  0000 C CNN
-F 2 "Capacitor_SMD:C_0402_1005Metric" H 10400 1950 50  0001 C CNN
+F 2 "Resistor_SMD:R_0402_1005Metric" H 10400 1950 50  0001 C CNN
 F 3 "~" H 10400 1950 50  0001 C CNN
 	1    10400 1950
@@
 F 0 "R21" V 10300 2300 50  0000 C CNN
 F 1 "33K" V 10400 2300 50  0000 C CNN
-F 2 "Capacitor_SMD:C_0402_1005Metric" H 10400 2300 50  0001 C CNN
+F 2 "Resistor_SMD:R_0402_1005Metric" H 10400 2300 50  0001 C CNN
 F 3 "~" H 10400 2300 50  0001 C CNN
 	1    10400 2300
@@
 F 0 "R17" V 8050 1350 50  0000 C CNN
 F 1 "33K" V 8150 1350 50  0000 C CNN
-F 2 "Capacitor_SMD:C_0402_1005Metric" H 8150 1350 50  0001 C CNN
+F 2 "Resistor_SMD:R_0402_1005Metric" H 8150 1350 50  0001 C CNN
 F 3 "~" H 8150 1350 50  0001 C CNN
 	1    8150 1350
@@
 Wire Wire Line
 	9950 4350 9950 4450
+$Comp
+L power:GNDA #PWR081
+U 1 1 61789D74
+P 1200 4650
+F 0 "#PWR081" H 1200 4400 50  0001 C CNN
+F 1 "GNDA" V 1205 4523 50  0000 R CNN
+F 2 "" H 1200 4650 50  0001 C CNN
+F 3 "" H 1200 4650 50  0001 C CNN
+	1    1200 4650
+	0    1    1    0
+$EndComp
+$Comp
+L power:GND #PWR082
+U 1 1 6178A5EB
+P 1600 4650
+F 0 "#PWR082" H 1600 4400 50  0001 C CNN
+F 1 "GND" V 1605 4522 50  0000 R CNN
+F 2 "" H 1600 4650 50  0001 C CNN
+F 3 "" H 1600 4650 50  0001 C CNN
+	1    1600 4650
+	0    -1   -1   0
+$EndComp
+$Comp
+L Device:R_Small R26
+U 1 1 6178B1AE
+P 1400 4650
+F 0 "R26" V 1450 4500 50  0000 C CNN
+F 1 "0R" V 1400 4650 50  0000 C CNN
+F 2 "Resistor_SMD:R_0402_1005Metric" H 1400 4650 50  0001 C CNN
+F 3 "~" H 1400 4650 50  0001 C CNN
+	1    1400 4650
+	0    -1   -1   0
+$EndComp
+Wire Wire Line
+	1500 4650 1600 4650
+Wire Wire Line
+	1300 4650 1200 4650
 $EndSCHEMATC
