File: SynthoGame/SynthoGame_bottom/TouchMatrix.sch (KiCad schematic (older format))
At the start: 21 parts, among them U7 AT42QT1244

Commit message: Removing touch from bottom board
Parts:
- removed C61, C62, C63: 4.7n, Capacitor_SMD:C_0402_1005Metric, symbol Device:C_Small
- removed C64, C65, C66: 100n, Capacitor_SMD:C_0402_1005Metric, symbol Device:C_Small
- removed R27, R28, R29, R30, R31, R32, R33, R34, R35, R36, R37, R38, R39, R40: 1K, Resistor_SMD:R_0402_1005Metric, symbol Device:R_Small
- removed U7: AT42QT1244, Package_QFP:TQFP-32_7x7mm_P0.8mm, symbol at42qt1244:AT42QT1244
Connections:
- net labels removed: +3.3V, A0, A1, CHANGE, DBG_CLK, GND, M_SYNC, RST, SCL, SDA, SMP, S_SYNC, X0, X1, X2, X3, X4, X5, X6, X7, Y0, Y1, Y2
- wire segments 74 -> 0

Commit message: Adding connector
Parts:
- added J9: Touch, Connector_PinSocket_2.54mm:PinSocket_2x06_P2.54mm_Vertical_SMD, symbol Connector_Generic:Conn_02x06_Odd_Even
Connections:
- new net 3V3: J9.10 (Pin_10)
- new net A0: J9.7 (Pin_7)
- new net A1: J9.9 (Pin_9)
- new net CHANGE: J9.6 (Pin_6)
- new net DBG_CLK: J9.8 (Pin_8)
- new net GND: J9.11 (Pin_11), J9.12 (Pin_12)
- new net M_SYNC: J9.2 (Pin_2)
- new net RST: J9.5 (Pin_5)
- new net SCL: J9.3 (Pin_3)
- new net SDA: J9.1 (Pin_1)
- new net S_SYNC: J9.4 (Pin_4)
Changed lines of the file:
@@
 Comment4 ""
 $EndDescr
+$Comp
+L Connector_Generic:Conn_02x06_Odd_Even J9
+U 1 1 61796D8D
+P 7200 3800
+F 0 "J9" H 7250 4217 50  0000 C CNN
+F 1 "Touch" H 7250 4126 50  0000 C CNN
+F 2 "Connector_PinSocket_2.54mm:PinSocket_2x06_P2.54mm_Vertical_SMD" H 7200 3800 50  0001 C CNN
+F 3 "~" H 7200 3800 50  0001 C CNN
+	1    7200 3800
+	1    0    0    -1
+$EndComp
+Text HLabel 6950 3600 0    50   BiDi ~ 0
+SDA
+Text HLabel 6950 3700 0    50   BiDi ~ 0
+SCL
+Text HLabel 6950 3800 0    50   Input ~ 0
+RST
+Text HLabel 6950 3900 0    50   Input ~ 0
+A0
+Text HLabel 6950 4000 0    50   Input ~ 0
+A1
+Text HLabel 7550 3600 2    50   Input ~ 0
+M_SYNC
+Text HLabel 7550 3700 2    50   Output ~ 0
+S_SYNC
+Text HLabel 7550 3800 2    50   Output ~ 0
+CHANGE
+Text HLabel 7550 3900 2    50   Output ~ 0
+DBG_CLK
+Text HLabel 7550 4000 2    50   Input ~ 0
+3V3
+Text HLabel 7550 4100 2    50   Input ~ 0
+GND
+Text HLabel 6950 4100 0    50   Input ~ 0
+GND
+Wire Wire Line
+	6950 3600 7000 3600
+Wire Wire Line
+	6950 3700 7000 3700
+Wire Wire Line
+	6950 3800 7000 3800
+Wire Wire Line
+	6950 3900 7000 3900
+Wire Wire Line
+	6950 4000 7000 4000
+Wire Wire Line
+	6950 4100 7000 4100
+Wire Wire Line
+	7500 3600 7550 3600
+Wire Wire Line
+	7500 3700 7550 3700
+Wire Wire Line
+	7500 3800 7550 3800
+Wire Wire Line
+	7500 3900 7550 3900
+Wire Wire Line
+	7500 4000 7550 4000
+Wire Wire Line
+	7500 4100 7550 4100
 $EndSCHEMATC
