File: SynthoGame/SynthoGame_bottom/SynthMIDI.sch (KiCad schematic (older format))
At the start: 9 parts, among them J6 JACK_TRS_6PINS_APPLE, J7 JACK_TRS_6PINS_APPLE, U5 TLP2361

Commit message: Routing
Connections:
- net MIDI_IN renamed IN_MIDI
- net MIDI_OUT renamed OUT_MIDI
Changed lines of the file:
@@
 Text GLabel 5300 4000 3    50   Input ~ 0
 GND
-Text GLabel 5900 3500 2    50   Input ~ 0
-MIDI_IN
 Wire Wire Line
 	4650 3350 4650 3300
@@
 Text GLabel 7000 2600 1    50   Input ~ 0
 +3V3
-Text GLabel 8550 4650 2    50   Input ~ 0
-MIDI_OUT
 $Comp
 L Device:D D4
@@
 Text HLabel 8550 4650 0    50   Output ~ 0
 OUT_MIDI
-Text GLabel 7250 4300 3    50   Input ~ 0
+Wire Wire Line
+	8550 4500 8700 4500
+Wire Wire Line
+	8550 4650 8700 4650
+Text Label 8700 4650 0    50   ~ 0
 MIDI_OUT
-Text GLabel 8550 4500 2    50   Input ~ 0
+Text Label 7250 4300 3    50   ~ 0
+MIDI_OUT
+Text Label 8700 4500 0    50   ~ 0
+MIDI_IN
+Text Label 5900 3500 0    50   ~ 0
 MIDI_IN
 $EndSCHEMATC

Commit message: resolve ERC errors, minor tweaks
Connections:
- no-connect marks 0 -> 7
Changed lines of the file:
@@
 Text Label 5900 3500 0    50   ~ 0
 MIDI_IN
+NoConn ~ 7600 3700
+NoConn ~ 6850 3050
+NoConn ~ 6950 3900
+NoConn ~ 3600 3750
+NoConn ~ 2800 3950
+NoConn ~ 2950 3950
+NoConn ~ 2850 3100
 $EndSCHEMATC
